File: Kicad/Versión_2/Etapa de filtro pasabajos/Etapa de filtro pasabajos.kicad_pcb (KiCad board)
At the start: 2 copper layers, 8 parts, among them J1 Conn_01x01_Pin, J15 Conn_01x01_Pin, J2 Conn_01x02_Pin, U5 TL082

Commit message: Fix: valores kicad
Parts:
- renumbered C20 to 1.5uF, R32 to 33kΩ, R31 to 33kΩ, C19 to 680nF
Changed lines of the file:
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@@
 		(descr "Resistor, Axial_DIN0207 series, Axial, Horizontal, pin pitch=10.16mm, 0.25W = 1/4W, length*diameter=6.3*2.5mm^2, http://cdn-reichelt.de/documents/datenblatt/B400/1_4W%23YAG.pdf")
 		(tags "Resistor Axial_DIN0207 series Axial Horizontal pin pitch 10.16mm 0.25W = 1/4W length 6.3mm diameter 2.5mm")
-		(property "Reference" "R32"
+		(property "Reference" "33kΩ"
 			(at 5.08 -2.37 0)
 			(layer "F.SilkS")
@@
 		(descr "C, Rect series, Radial, pin pitch=22.50mm, length*width=24*10.1mm^2, Capacitor, https://en.tdk.eu/inf/20/20/db/fc_2009/MKT_B32560_564.pdf")
 		(tags "C Rect series Radial pin pitch 22.50mm length 24mm width 10.1mm Capacitor")
-		(property "Reference" "C20"
+		(property "Reference" "1.5uF"
 			(at 11.25 -6.3 90)
 			(layer "F.SilkS")
@@
 		(descr "C, Rect series, Radial, pin pitch=7.50mm, length*width=10*2.5mm^2, Capacitor, http://www.wima.com/EN/WIMA_MKS_4.pdf")
 		(tags "C Rect series Radial pin pitch 7.50mm length 10mm width 2.5mm Capacitor")
-		(property "Reference" "C19"
+		(property "Reference" "680nF"
 			(at 3.75 -2.5 0)
 			(layer "F.SilkS")
@@
 		(descr "Resistor, Axial_DIN0207 series, Axial, Horizontal, pin pitch=10.16mm, 0.25W = 1/4W, length*diameter=6.3*2.5mm^2, http://cdn-reichelt.de/documents/datenblatt/B400/1_4W%23YAG.pdf")
 		(tags "Resistor Axial_DIN0207 series Axial Horizontal pin pitch 10.16mm 0.25W = 1/4W length 6.3mm diameter 2.5mm")
-		(property "Reference" "R31"
+		(property "Reference" "33kΩ"
 			(at 5.08 -2.37 0)
 			(layer "F.SilkS")
@@
 	)
 	(segment
+		(start 142.25 68)
+		(end 126 68)
+		(width 1.3)
+		(layer "B.Cu")
+		(net "Net-(J15-Pin_1)")
+	)
+	(segment
+		(start 129.88 78)
+		(end 130 78.12)
+		(width 1.3)
+		(layer "B.Cu")
+		(net "Net-(J15-Pin_1)")
+	)
+	(segment
+		(start 125.12 78.12)
+		(end 130 78.12)
+		(width 1.3)
+		(layer "B.Cu")
+		(net "Net-(J15-Pin_1)")
+	)
+	(segment
+		(start 124 77)
+		(end 124 79)
+		(width 1.3)
+		(layer "B.Cu")
+		(net "Net-(J15-Pin_1)")
+	)
+	(segment
+		(start 125.12 78.12)
+		(end 124.88 78.12)
+		(width 1.3)
+		(layer "B.Cu")
+		(net "Net-(J15-Pin_1)")
+	)
+	(segment
+		(start 124.88 78.12)
+		(end 124 79)
+		(width 1.3)
+		(layer "B.Cu")
+		(net "Net-(J15-Pin_1)")
+	)
+	(segment
+		(start 145 70.75)
+		(end 142.25 68)
+		(width 1.3)
+		(layer "B.Cu")
+		(net "Net-(J15-Pin_1)")
+	)
+	(segment
+		(start 124 70)
+		(end 124 77)
+		(width 1.3)
+		(layer "B.Cu")
+		(net "Net-(J15-Pin_1)")
+	)
+	(segment
+		(start 124 79)
+		(end 124 82.5)
+		(width 1.3)
+		(layer "B.Cu")
+		(net "Net-(J15-Pin_1)")
+	)
+	(segment
+		(start 126 68)
+		(end 124 70)
+		(width 1.3)
+		(layer "B.Cu")
+		(net "Net-(J15-Pin_1)")
+	)
+	(segment
+		(start 124 82.5)
+		(end 124.5 83)
+		(width 1.3)
+		(layer "B.Cu")
+		(net "Net-(J15-Pin_1)")
+	)
+	(segment
+		(start 130 78.12)
+		(end 132.54 78.12)
+		(width 1.3)
+		(layer "B.Cu")
+		(net "Net-(J15-Pin_1)")
+	)
+	(segment
+		(start 124 77)
+		(end 125.12 78.12)
+		(width 1.3)
+		(layer "B.Cu")
+		(net "Net-(J15-Pin_1)")
+	)
+	(segment
 		(start 135.08 78.12)
 		(end 132.7 80.5)
@@
 	)
 	(segment
-		(start 142.25 68)
-		(end 126 68)
-		(width 1.3)
-		(layer "B.Cu")
-		(net "Net-(J15-Pin_1)")
-	)
-	(segment
-		(start 129.88 78)
-		(end 130 78.12)
-		(width 1.3)
-		(layer "B.Cu")
-		(net "Net-(J15-Pin_1)")
-	)
-	(segment
-		(start 125.12 78.12)
-		(end 130 78.12)
-		(width 1.3)
-		(layer "B.Cu")
-		(net "Net-(J15-Pin_1)")
-	)
-	(segment
-		(start 124 77)
-		(end 124 79)
-		(width 1.3)
-		(layer "B.Cu")
-		(net "Net-(J15-Pin_1)")
-	)
-	(segment
-		(start 125.12 78.12)
-		(end 124.88 78.12)
-		(width 1.3)
-		(layer "B.Cu")
-		(net "Net-(J15-Pin_1)")
-	)
-	(segment
-		(start 124.88 78.12)
-		(end 124 79)
-		(width 1.3)
-		(layer "B.Cu")
-		(net "Net-(J15-Pin_1)")
-	)
-	(segment
-		(start 145 70.75)
-		(end 142.25 68)
-		(width 1.3)
-		(layer "B.Cu")
-		(net "Net-(J15-Pin_1)")
-	)
-	(segment
-		(start 124 70)
-		(end 124 77)
-		(width 1.3)
-		(layer "B.Cu")
-		(net "Net-(J15-Pin_1)")
-	)
-	(segment
-		(start 124 79)
-		(end 124 82.5)
-		(width 1.3)
-		(layer "B.Cu")
-		(net "Net-(J15-Pin_1)")
-	)
-	(segment
-		(start 126 68)
-		(end 124 70)
-		(width 1.3)
-		(layer "B.Cu")
-		(net "Net-(J15-Pin_1)")
-	)
-	(segment
-		(start 124 82.5)
-		(end 124.5 83)
-		(width 1.3)
-		(layer "B.Cu")
-		(net "Net-(J15-Pin_1)")
-	)
-	(segment
-		(start 130 78.12)
-		(end 132.54 78.12)
-		(width 1.3)
-		(layer "B.Cu")
-		(net "Net-(J15-Pin_1)")
-	)
-	(segment
-		(start 124 77)
-		(end 125.12 78.12)
-		(width 1.3)
-		(layer "B.Cu")
-		(net "Net-(J15-Pin_1)")
+		(start 137.62 76.62)
+		(end 137.62 78.12)
+		(width 1.3)
+		(layer "B.Cu")
+		(net "Net-(J2-Pin_2)")
+	)
+	(segment
+		(start 136.315 75.315)
+		(end 137.62 76.62)
+		(width 1.3)
+		(layer "B.Cu")
+		(net "Net-(J2-Pin_2)")
+	)
+	(segment
+		(start 126.5 75.315)
+		(end 136.315 75.315)
+		(width 1.3)
+		(layer "B.Cu")
+		(net "Net-(J2-Pin_2)")
+	)
+	(segment
+		(start 128.685 73.315)
+		(end 130 72)
+		(width 1.3)
+		(layer "B.Cu")
+		(net "Net-(J2-Pin_1)")
+	)
+	(segment
+		(start 126.5 73.315)
+		(end 128.685 73.315)
+		(width 1.3)
+		(layer "B.Cu")
+		(net "Net-(J2-Pin_1)")
+	)
+	(segment
+		(start 130 72)
+		(end 130 70.5)
+		(width 1.3)
+		(layer "B.Cu")
+		(net "Net-(J2-Pin_1)")
 	)
 	(segment
@@
 		(net "Net-(J1-Pin_1)")
 	)
-	(segment
-		(start 137.62 76.62)
-		(end 137.62 78.12)
-		(width 1.3)
-		(layer "B.Cu")
-		(net "Net-(J2-Pin_2)")
-	)
-	(segment
-		(start 136.315 75.315)
-		(end 137.62 76.62)
-		(width 1.3)
-		(layer "B.Cu")
-		(net "Net-(J2-Pin_2)")
-	)
-	(segment
-		(start 126.5 75.315)
-		(end 136.315 75.315)
-		(width 1.3)
-		(layer "B.Cu")
-		(net "Net-(J2-Pin_2)")
-	)
-	(segment
-		(start 128.685 73.315)
-		(end 130 72)
-		(width 1.3)
-		(layer "B.Cu")
-		(net "Net-(J2-Pin_1)")
-	)
-	(segment
-		(start 126.5 73.315)
-		(end 128.685 73.315)
-		(width 1.3)
-		(layer "B.Cu")
-		(net "Net-(J2-Pin_1)")
-	)
-	(segment
-		(start 130 72)
-		(end 130 70.5)
-		(width 1.3)
-		(layer "B.Cu")
-		(net "Net-(J2-Pin_1)")
-	)
 	(zone
