File: Kicad/Versión_2/Etapa de rectificación de presición/Etapa de rectificación de presición.kicad_pcb (KiCad board)
At the start: 2 copper layers, 11 parts, among them J1 Conn_01x02_Pin, J2 Conn_01x01_Pin, J3 Conn_01x01_Pin, U4 TL084

Commit message: Fix: valores kicad
Parts:
- renumbered R24 to 10kΩ, R22 to 10kΩ, R21 to 10kΩ, R25 to 10kΩ, R23 to 10kΩ
