File: Kicad/Versión_2/Etapa de filtro pasabanda/Etapa de filtro pasabanda.kicad_pcb (KiCad board)
At the start: 2 copper layers, 23 parts, among them J1 Conn_01x01_Pin, J2 Conn_01x04_Pin, J5 Conn_01x02_Pin, U1 AD620, U2 TL084

Commit message: Fix: valores kicad
Parts:
- 47nF: renamed from C1; value C -> 47nf
- renumbered C7 to 1.5nF, R9 to 100kΩ, R3 to 100Ω, R6 to 10kΩ, R5 to 10kΩ, R4 to 120kΩ, R8 to 12kΩ, R7 to 180kΩ, C8 to 3.3nF, C3 to 39nF, C6 to 39nF, C5 to 4.7nF, C2 to 4.7nF, R1 to 470Ω, C4 to 47nF, R10 to 5.1kΩ, R2 to 68kΩ
Changed lines of the file:
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@@
 		(descr "C, Rect series, Radial, pin pitch=7.50mm, length*width=10*2.5mm^2, Capacitor, http://www.wima.com/EN/WIMA_MKS_4.pdf")
 		(tags "C Rect series Radial pin pitch 7.50mm length 10mm width 2.5mm Capacitor")
-		(property "Reference" "C1"
+		(property "Reference" "47nF"
 			(at 3.75 -2.5 0)
 			(layer "F.SilkS")
@@
 			)
 		)
-		(property "Value" "C"
+		(property "Value" "47nf"
 			(at 3.75 2.5 0)
 			(layer "F.Fab")
@@
 		(descr "C, Rect series, Radial, pin pitch=7.50mm, length*width=10*2.5mm^2, Capacitor, http://www.wima.com/EN/WIMA_MKS_4.pdf")
 		(tags "C Rect series Radial pin pitch 7.50mm length 10mm width 2.5mm Capacitor")
-		(property "Reference" "C4"
+		(property "Reference" "47nF"
 			(at 3.75 -2.5 0)
 			(layer "F.SilkS")
@@
 		(descr "C, Rect series, Radial, pin pitch=7.50mm, length*width=10*2.5mm^2, Capacitor, http://www.wima.com/EN/WIMA_MKS_4.pdf")
 		(tags "C Rect series Radial pin pitch 7.50mm length 10mm width 2.5mm Capacitor")
-		(property "Reference" "C3"
+		(property "Reference" "39nF"
 			(at 3.75 -2.5 0)
 			(layer "F.SilkS")
@@
 		(descr "Resistor, Axial_DIN0207 series, Axial, Horizontal, pin pitch=10.16mm, 0.25W = 1/4W, length*diameter=6.3*2.5mm^2, http://cdn-reichelt.de/documents/datenblatt/B400/1_4W%23YAG.pdf")
 		(tags "Resistor Axial_DIN0207 series Axial Horizontal pin pitch 10.16mm 0.25W = 1/4W length 6.3mm diameter 2.5mm")
-		(property "Reference" "R8"
+		(property "Reference" "12kΩ"
 			(at 5.08 -2.37 0)
 			(layer "F.SilkS")
@@
 		(descr "Resistor, Axial_DIN0207 series, Axial, Horizontal, pin pitch=10.16mm, 0.25W = 1/4W, length*diameter=6.3*2.5mm^2, http://cdn-reichelt.de/documents/datenblatt/B400/1_4W%23YAG.pdf")
 		(tags "Resistor Axial_DIN0207 series Axial Horizontal pin pitch 10.16mm 0.25W = 1/4W length 6.3mm diameter 2.5mm")
-		(property "Reference" "R7"
+		(property "Reference" "180kΩ"
 			(at 5.08 -2.37 0)
 			(layer "F.SilkS")
@@
 		(descr "Resistor, Axial_DIN0207 series, Axial, Horizontal, pin pitch=10.16mm, 0.25W = 1/4W, length*diameter=6.3*2.5mm^2, http://cdn-reichelt.de/documents/datenblatt/B400/1_4W%23YAG.pdf")
 		(tags "Resistor Axial_DIN0207 series Axial Horizontal pin pitch 10.16mm 0.25W = 1/4W length 6.3mm diameter 2.5mm")
-		(property "Reference" "R4"
+		(property "Reference" "120kΩ"
 			(at 5.08 -2.37 0)
 			(layer "F.SilkS")
@@
 		(descr "C, Rect series, Radial, pin pitch=7.50mm, length*width=10*2.5mm^2, Capacitor, http://www.wima.com/EN/WIMA_MKS_4.pdf")
 		(tags "C Rect series Radial pin pitch 7.50mm length 10mm width 2.5mm Capacitor")
-		(property "Reference" "C5"
+		(property "Reference" "4.7nF"
 			(at 3.75 -2.5 0)
 			(layer "F.SilkS")
@@
 		(descr "C, Rect series, Radial, pin pitch=7.50mm, length*width=10*2.5mm^2, Capacitor, http://www.wima.com/EN/WIMA_MKS_4.pdf")
 		(tags "C Rect series Radial pin pitch 7.50mm length 10mm width 2.5mm Capacitor")
-		(property "Reference" "C2"
+		(property "Reference" "4.7nF"
 			(at 3.75 -2.5 0)
 			(layer "F.SilkS")
@@
 		(descr "Resistor, Axial_DIN0207 series, Axial, Horizontal, pin pitch=10.16mm, 0.25W = 1/4W, length*diameter=6.3*2.5mm^2, http://cdn-reichelt.de/documents/datenblatt/B400/1_4W%23YAG.pdf")
 		(tags "Resistor Axial_DIN0207 series Axial Horizontal pin pitch 10.16mm 0.25W = 1/4W length 6.3mm diameter 2.5mm")
-		(property "Reference" "R6"
+		(property "Reference" "10kΩ"
 			(at 5.08 -2.37 0)
 			(layer "F.SilkS")
@@
 		(descr "C, Rect series, Radial, pin pitch=7.50mm, length*width=10*2.5mm^2, Capacitor, http://www.wima.com/EN/WIMA_MKS_4.pdf")
 		(tags "C Rect series Radial pin pitch 7.50mm length 10mm width 2.5mm Capacitor")
-		(property "Reference" "C8"
+		(property "Reference" "3.3nF"
 			(at 3.75 -2.5 0)
 			(layer "F.SilkS")
@@
 		(descr "C, Rect series, Radial, pin pitch=7.50mm, length*width=10*2.5mm^2, Capacitor, http://www.wima.com/EN/WIMA_MKS_4.pdf")
 		(tags "C Rect series Radial pin pitch 7.50mm length 10mm width 2.5mm Capacitor")
-		(property "Reference" "C6"
+		(property "Reference" "39nF"
 			(at 3.75 -2.5 0)
 			(layer "F.SilkS")
@@
 		(descr "Resistor, Axial_DIN0207 series, Axial, Horizontal, pin pitch=10.16mm, 0.25W = 1/4W, length*diameter=6.3*2.5mm^2, http://cdn-reichelt.de/documents/datenblatt/B400/1_4W%23YAG.pdf")
 		(tags "Resistor Axial_DIN0207 series Axial Horizontal pin pitch 10.16mm 0.25W = 1/4W length 6.3mm diameter 2.5mm")
-		(property "Reference" "R3"
+		(property "Reference" "100Ω"
 			(at 5.08 -2.37 0)
 			(layer "F.SilkS")
@@
 		(descr "Resistor, Axial_DIN0207 series, Axial, Horizontal, pin pitch=10.16mm, 0.25W = 1/4W, length*diameter=6.3*2.5mm^2, http://cdn-reichelt.de/documents/datenblatt/B400/1_4W%23YAG.pdf")
 		(tags "Resistor Axial_DIN0207 series Axial Horizontal pin pitch 10.16mm 0.25W = 1/4W length 6.3mm diameter 2.5mm")
-		(property "Reference" "R5"
+		(property "Reference" "10kΩ"
 			(at 5.08 -2.37 0)
 			(layer "F.SilkS")
@@
 		(descr "Resistor, Axial_DIN0207 series, Axial, Horizontal, pin pitch=10.16mm, 0.25W = 1/4W, length*diameter=6.3*2.5mm^2, http://cdn-reichelt.de/documents/datenblatt/B400/1_4W%23YAG.pdf")
 		(tags "Resistor Axial_DIN0207 series Axial Horizontal pin pitch 10.16mm 0.25W = 1/4W length 6.3mm diameter 2.5mm")
-		(property "Reference" "R2"
+		(property "Reference" "68kΩ"
 			(at 5.08 -2.37 0)
 			(layer "F.SilkS")
@@
 		(descr "C, Rect series, Radial, pin pitch=7.50mm, length*width=10*2.5mm^2, Capacitor, http://www.wima.com/EN/WIMA_MKS_4.pdf")
 		(tags "C Rect series Radial pin pitch 7.50mm length 10mm width 2.5mm Capacitor")
-		(property "Reference" "C7"
+		(property "Reference" "1.5nF"
 			(at 3.75 -2.5 0)
 			(layer "F.SilkS")
@@
 		(descr "Resistor, Axial_DIN0207 series, Axial, Horizontal, pin pitch=10.16mm, 0.25W = 1/4W, length*diameter=6.3*2.5mm^2, http://cdn-reichelt.de/documents/datenblatt/B400/1_4W%23YAG.pdf")
 		(tags "Resistor Axial_DIN0207 series Axial Horizontal pin pitch 10.16mm 0.25W = 1/4W length 6.3mm diameter 2.5mm")
-		(property "Reference" "R9"
+		(property "Reference" "100kΩ"
 			(at 5.08 -2.37 0)
 			(layer "F.SilkS")
@@
 		(descr "Resistor, Axial_DIN0207 series, Axial, Horizontal, pin pitch=10.16mm, 0.25W = 1/4W, length*diameter=6.3*2.5mm^2, http://cdn-reichelt.de/documents/datenblatt/B400/1_4W%23YAG.pdf")
 		(tags "Resistor Axial_DIN0207 series Axial Horizontal pin pitch 10.16mm 0.25W = 1/4W length 6.3mm diameter 2.5mm")
-		(property "Reference" "R1"
+		(property "Reference" "470Ω"
 			(at 5.08 -2.37 90)
 			(layer "F.SilkS")
@@
 		(descr "Resistor, Axial_DIN0207 series, Axial, Horizontal, pin pitch=10.16mm, 0.25W = 1/4W, length*diameter=6.3*2.5mm^2, http://cdn-reichelt.de/documents/datenblatt/B400/1_4W%23YAG.pdf")
 		(tags "Resistor Axial_DIN0207 series Axial Horizontal pin pitch 10.16mm 0.25W = 1/4W length 6.3mm diameter 2.5mm")
-		(property "Reference" "R10"
+		(property "Reference" "5.1kΩ"
 			(at 5.08 -2.37 0)
 			(layer "F.SilkS")

Commit message: fix/FG/KiCad_PCB
Parts:
- renumbered 180kΩ to 100kΩ, 5.1kΩ to 12kΩ, 100kΩ to 180kΩ, 12kΩ to 5.6kΩ
Changed lines of the file:
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@@
 		(descr "Resistor, Axial_DIN0207 series, Axial, Horizontal, pin pitch=10.16mm, 0.25W = 1/4W, length*diameter=6.3*2.5mm^2, http://cdn-reichelt.de/documents/datenblatt/B400/1_4W%23YAG.pdf")
 		(tags "Resistor Axial_DIN0207 series Axial Horizontal pin pitch 10.16mm 0.25W = 1/4W length 6.3mm diameter 2.5mm")
-		(property "Reference" "12kΩ"
+		(property "Reference" "5.6kΩ"
 			(at 5.08 -2.37 0)
 			(layer "F.SilkS")
@@
 		(descr "Resistor, Axial_DIN0207 series, Axial, Horizontal, pin pitch=10.16mm, 0.25W = 1/4W, length*diameter=6.3*2.5mm^2, http://cdn-reichelt.de/documents/datenblatt/B400/1_4W%23YAG.pdf")
 		(tags "Resistor Axial_DIN0207 series Axial Horizontal pin pitch 10.16mm 0.25W = 1/4W length 6.3mm diameter 2.5mm")
-		(property "Reference" "180kΩ"
+		(property "Reference" "100kΩ"
 			(at 5.08 -2.37 0)
 			(layer "F.SilkS")
@@
 		(descr "Resistor, Axial_DIN0207 series, Axial, Horizontal, pin pitch=10.16mm, 0.25W = 1/4W, length*diameter=6.3*2.5mm^2, http://cdn-reichelt.de/documents/datenblatt/B400/1_4W%23YAG.pdf")
 		(tags "Resistor Axial_DIN0207 series Axial Horizontal pin pitch 10.16mm 0.25W = 1/4W length 6.3mm diameter 2.5mm")
-		(property "Reference" "100kΩ"
+		(property "Reference" "180kΩ"
 			(at 5.08 -2.37 0)
 			(layer "F.SilkS")
@@
 		(descr "Resistor, Axial_DIN0207 series, Axial, Horizontal, pin pitch=10.16mm, 0.25W = 1/4W, length*diameter=6.3*2.5mm^2, http://cdn-reichelt.de/documents/datenblatt/B400/1_4W%23YAG.pdf")
 		(tags "Resistor Axial_DIN0207 series Axial Horizontal pin pitch 10.16mm 0.25W = 1/4W length 6.3mm diameter 2.5mm")
-		(property "Reference" "5.1kΩ"
+		(property "Reference" "12kΩ"
 			(at 5.08 -2.37 0)
 			(layer "F.SilkS")
