File: Kicad/Versión_1/PCB_etapa_analógica.kicad_sch (KiCad schematic)
At the start: 44 parts, among them J1 Conn_01x01_Pin, J12 Conn_01x01_Pin, J13 Conn_01x01_Pin, J14 Conn_01x01_Pin, J15 Conn_01x01_Pin, J2 Conn_01x01_Pin, J3 Conn_01x01_Pin, J4 Conn_01x01_Pin, J5 Conn_01x01_Pin, J6 Conn_01x01_Pin, J7 Conn_01x01_Pin, U1 AD620, U2 TL084, U4 TL084, U5 TL082

Commit message: feat(modelos): Añado modelo final de la ortesis
Parts:
- removed C19, C20: C, Capacitor_THT:C_Rect_L10.0mm_W2.5mm_P7.50mm_MKS4, symbol Device:C
- removed D1, D2: D, Diode_THT:D_DO-41_SOD81_P10.16mm_Horizontal, symbol Device:D
- removed J1, J12, J13, J14, J15, J2, J3, J5, J6, J7: Conn_01x01_Pin, Connector_PinHeader_1.00mm:PinHeader_1x01_P1.00mm_Vertical, symbol Connector:Conn_01x01_Pin
- removed R21, R22, R23, R24, R25, R31, R32: R, Resistor_THT:R_Axial_DIN0207_L6.3mm_D2.5mm_P10.16mm_Horizontal, symbol Device:R
- removed U4: TL084, Package_DIP:DIP-14_W7.62mm_LongPads, symbol Amplifier_Operational:TL084
- removed U5: TL082, Package_DIP:DIP-8_W7.62mm, symbol Amplifier_Operational:TL082
- added J1, J2, J3: Conn_01x02_Pin, Connector_PinHeader_2.00mm:PinHeader_1x02_P2.00mm_Vertical, symbol Connector:Conn_01x02_Pin
- C1, C2, C3, C4, C5, C6, C7, C8: footprint Capacitor_THT:C_Rect_L10.0mm_W2.5mm_P7.50mm_MKS4 -> Capacitor_THT:C_Disc_D6.0mm_W2.5mm_P5.00mm
- J4: footprint Connector_PinHeader_1.00mm:PinHeader_1x01_P1.00mm_Vertical -> Connector_PinHeader_2.00mm:PinHeader_1x01_P2.00mm_Vertical
Connections:
- net at U1.2 (-): now also J1.1 (Pin_1)
- net at U1.3 (+): now also J1.2 (Pin_2); no longer J4.1 (Pin_1)
- net at U1.4 (Vs-): now also J2.2 (Pin_2)
- net at U1.7 (Vs+): now also J2.1 (Pin_1)
- net at C8.1, U2.5 (+), U2.7: now also J4.1 (Pin_1)
- net at U2.11 (V-): now also J3.2 (Pin_2)
- net at U2.4 (V+): now also J3.1 (Pin_1)
Other:
- moved on the sheet: C1, C2, C3, C4, C5, C6, C7, C8, R1, R10, R2, R3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
